Commit message: increasing default clearance

File: ur_description/urdf/ur5_robot.urdf.xacro (robot description, xacro)
@@ -12,5 +12,5 @@
     <parent link="world" />
     <child link = "base_link" />
-    <origin xyz="0.0 0.0 0.0" rpy="0.0 0.0 0.0" />
+    <origin xyz="0.0 0.0 0.1" rpy="0.0 0.0 0.0" />
   </joint>
 </robot>
